Commit message: Fixed issues with loading the robots

File: four_wheel_robot/description/robot_core.xacro (robot description, xacro)
@@ -14,8 +14,8 @@
     </material>
     <!-- Base link -->
-    <link name="dummy">
+    <link name="ground">
     </link>
     <joint name="chassis_joint" type="fixed">
-        <parent link="dummy"/>
+        <parent link="ground"/>
         <child link="base_link"/>
         <origin xyz="0.0 0 0" rpy="0 0 0"/>
