Commit message: added front and rear lidars to the robot

File: mobile_manipulator/description/robot.urdf.xacro (robot description, xacro)
@@ -2,3 +2,5 @@
 <robot xmlns:xacro="http://www.ros.org/wiki/xacro" name="robot">
     <xacro:include filename="robot_core.xacro"/>
+    <xacro:include filename="sensors/lidars.xacro"/>
+    <xacro:include filename="gazebo_control.xacro"/>
 </robot>

File: mobile_manipulator/description/robot_core.xacro (robot description, xacro)
@@ -1,11 +1,4 @@
 <?xml version="1.0"?>
 <robot xmlns:xacro="http://www.ros.org/wiki/xacro" name="robot">
-    <link name="ground">
-    </link>
-    <joint name="ground_link" type="fixed">
-        <parent link="ground"/>
-        <child link="cart"/>
-        <origin xyz="0 0 0.18" rpy="0 0 0"/>
-    </joint>
     <link name="cart">
         <inertial>
@@ -62,4 +55,6 @@
     <gazebo reference="front_right_wheel">
         <material>Gazebo/Black</material>
+        <mu1 value="0.001"></mu1>
+        <mu2 value="0.001"></mu2>
     </gazebo>
     <!--Rear right wheel-->
@@ -91,4 +86,6 @@
     <gazebo reference="rear_right_wheel">
         <material>Gazebo/Black</material>
+        <mu1 value="0.001"></mu1>
+        <mu2 value="0.001"></mu2>
     </gazebo>
     <!--Front left wheel-->
@@ -120,4 +117,6 @@
     <gazebo reference="front_left_wheel">
         <material>Gazebo/Black</material>
+        <mu1 value="0.001"></mu1>
+        <mu2 value="0.001"></mu2>
     </gazebo>
     <!-- Rear left wheel -->
@@ -149,4 +148,6 @@
     <gazebo reference="rear_left_wheel">
         <material>Gazebo/Black</material>
+        <mu1 value="0.001"></mu1>
+        <mu2 value="0.001"></mu2>
     </gazebo>
 </robot>

File: mobile_manipulator/description/sensors/lidars.xacro (robot description, xacro)
@@ -1,3 +1,113 @@
 <?xml version="1.0"?>
 <robot xmlns:xacro="http://www.ros.org/wiki/xacro" name="robot">
+    <!-- Front Lidar -->
+    <joint name="front_lidar_joint" type="fixed">
+        <origin xyz="0.0 -0.115682 -0.08" rpy="0 0 0"/>
+        <parent link="cart"/>
+        <child link="front_lidar"/>
+    </joint>
+    <link name="front_lidar">
+        <inertial>
+            <origin xyz="-4.736301440343586e-17 1.8181818177420705e-07 0.012499999999999983" rpy="0 0 0"/>
+            <mass value="0.18881462721926778"/>
+            <inertia ixx="2.4e-05" iyy="2.4e-05" izz="2.9e-05" ixy="-0.0" iyz="0.0" ixz="-0.0"/>
+        </inertial>
+        <visual>
+            <origin xyz="0.0 0.115682 0.08" rpy="0 0 0"/>
+            <geometry>
+            <mesh filename="file://$(find mobile_manipulator)/meshes/lidar_front.stl" scale="0.001 0.001 0.001"/>
+            </geometry>
+        </visual>
+        <collision>
+            <origin xyz="0.0 0.115682 0.08" rpy="0 0 0"/>
+            <geometry>
+            <mesh filename="file://$(find mobile_manipulator)/meshes/lidar_front.stl" scale="0.001 0.001 0.001"/>
+            </geometry>
+        </collision>
+    </link>
+    <gazebo reference="front_lidar">
+        <material>Gazebo/Red</material>
+        <sensor type="ray" name="front_lidar">
+            <pose>0 0 0 0 0 0</pose>
+            <visualize>true</visualize>
+            <update_rate>10</update_rate>
+            <ray>
+                <scan>
+                    <horizontal>
+                        <samples>360</samples>
+                        <resolution>1</resolution>
+                        <min_angle>0.2</min_angle>
+                        <max_angle>2.9</max_angle>
+                    </horizontal>
+                </scan>
+                <range>
+                    <min>0.3</min>
+                    <max>6</max>
+                    <resolution>0.01</resolution>
+                </range>
+            </ray>
+            <plugin name="lidar_controller_front" filename="libgazebo_ros_ray_sensor.so">
+                <ros>
+                    <argument>--ros-args --remap ~/out:=front_lidar_scan</argument>
+                </ros>
+                <output_type>sensor_msgs/LaserScan</output_type>
+                <frame_name>front_lidar</frame_name>
+            </plugin>
+        </sensor>
+    </gazebo>
+    <!-- Rear Lidar -->
+    <joint name="rear_lidar_joint" type="fixed">
+        <origin xyz="0.0 -1.274318 -0.08" rpy="0 0 0"/>
+        <parent link="cart"/>
+        <child link="rear_lidar"/>
+    </joint>
+    <link name="rear_lidar">
+        <inertial>
+            <origin xyz="1.4803623793059169e-16 -1.81818181843596e-07 0.012499999999999914" rpy="0 0 0"/>
+            <mass value="0.18881462721926778"/>
+            <inertia ixx="2.4e-05" iyy="2.4e-05" izz="2.9e-05" ixy="-0.0" iyz="0.0" ixz="-0.0"/>
+        </inertial>
+        <visual>
+            <origin xyz="-0.0 1.274318 0.08" rpy="0 0 0"/>
+            <geometry>
+            <mesh filename="file://$(find mobile_manipulator)/meshes/lidar_rear.stl" scale="0.001 0.001 0.001"/>
+            </geometry>
+        </visual>
+        <collision>
+            <origin xyz="-0.0 1.274318 0.08" rpy="0 0 0"/>
+            <geometry>
+            <mesh filename="file://$(find mobile_manipulator)/meshes/lidar_rear.stl" scale="0.001 0.001 0.001"/>
+            </geometry>
+        </collision>
+    </link>
+    <gazebo reference="rear_lidar">
+        <material>Gazebo/Red</material>
+        <sensor type="ray" name="rear_lidar">
+            <pose>0 0 0 0 0 0</pose>
+            <visualize>true</visualize>
+            <update_rate>10</update_rate>
+            <ray>
+                <scan>
+                    <horizontal>
+                        <samples>360</samples>
+                        <resolution>1</resolution>
+                        <min_angle>-0.2</min_angle>
+                        <max_angle>-2.9</max_angle>
+                    </horizontal>
+                </scan>
+                <range>
+                    <min>0.3</min>
+                    <max>6</max>
+                    <resolution>0.01</resolution>
+                </range>
+            </ray>
+            <plugin name="lidar_controller_rear" filename="libgazebo_ros_ray_sensor.so">
+                <ros>
+                    <argument>--ros-args --remap ~/out:=rear_lidar_scan</argument>
+                </ros>
+                <output_type>sensor_msgs/LaserScan</output_type>
+                <frame_name>rear_lidar</frame_name>
+            </plugin>
+        </sensor>
+    </gazebo>
 </robot>

Commit message: removed gazebo plannar drive plugin

File: mobile_manipulator/description/robot.urdf.xacro (robot description, xacro)
@@ -3,4 +3,4 @@
     <xacro:include filename="robot_core.xacro"/>
     <xacro:include filename="sensors/lidars.xacro"/>
-    <xacro:include filename="gazebo_control.xacro"/>
+    <xacro:include filename="sensors/cameras.xacro"/>
 </robot>

File: mobile_manipulator/description/robot_core.xacro (robot description, xacro)
@@ -1,4 +1,11 @@
 <?xml version="1.0"?>
 <robot xmlns:xacro="http://www.ros.org/wiki/xacro" name="robot">
+    <joint name="ground_link" type="fixed">
+        <parent link="ground"/>
+        <child link="cart"/>
+        <origin xyz="0 0 0.18" rpy="0 0 0"/>
+    </joint>
+    <link name="ground">
+    </link>
     <link name="cart">
         <inertial>
@@ -151,3 +158,31 @@
         <mu2 value="0.001"></mu2>
     </gazebo>
+    <!--Basket-->
+    <joint name="basket_joint" type="fixed">
+        <origin xyz="0.0 -0.765223 0.6" rpy="0 0 0"/>
+        <parent link="cart"/>
+        <child link="basket_link"/>
+    </joint>
+    <link name="basket_link">
+        <inertial>
+            <origin xyz="0.0003367874890503231 -0.0009035016282807895 0.04026929343329555" rpy="0 0 0"/>
+            <mass value="235.5335761839034"/>
+            <inertia ixx="51.392071" iyy="12.587293" izz="62.459782" ixy="1.059027" iyz="0.016958" ixz="-0.006325"/>
+        </inertial>
+        <visual>
+            <origin xyz="-0.0 0.765223 -0.6" rpy="0 0 0"/>
+            <geometry>
+            <mesh filename="file://$(find mobile_manipulator)/meshes/basket.stl" scale="0.001 0.001 0.001"/>
+            </geometry>
+        </visual>
+        <collision>
+            <origin xyz="-0.0 0.765223 -0.6" rpy="0 0 0"/>
+            <geometry>
+            <mesh filename="file://$(find mobile_manipulator)/meshes/basket.stl" scale="0.001 0.001 0.001"/>
+            </geometry>
+        </collision>
+    </link>
+    <gazebo reference="basket_link">
+        <material>Gazebo/Yellow</material>
+    </gazebo>
 </robot>

Commit message: addded manipulators

File: mobile_manipulator/description/robot.urdf.xacro (robot description, xacro)
@@ -2,4 +2,5 @@
 <robot xmlns:xacro="http://www.ros.org/wiki/xacro" name="robot">
     <xacro:include filename="robot_core.xacro"/>
+    <xacro:include filename="robot_arm.xacro"/>
     <xacro:include filename="sensors/lidars.xacro"/>
     <xacro:include filename="sensors/cameras.xacro"/>

File: mobile_manipulator/description/robot_core.xacro (robot description, xacro)
@@ -31,5 +31,5 @@
     </link>
     <gazebo reference="cart">
-        <material>Gazebo/Grey</material>
+        <material>Gazebo/DarkGrey</material>
     </gazebo>
     <!--Wheels-->
