Commit message: added images

File: mobile_manipulator/description/robot_arm.xacro (robot description, xacro)
@@ -2,5 +2,5 @@
 <robot xmlns:xacro="http://www.ros.org/wiki/xacro" name="robot">
     <!--Arm Base One-->
-    <joint name="arm_one_base_joint" type="continuous">
+    <joint name="arm_one_base_joint" type="fixed">
         <origin xyz="0.275 -0.675 0.07" rpy="0 0 0"/>
         <parent link="basket_link"/>
@@ -31,5 +31,5 @@
     </gazebo>
     <!--Arm One Link-1-->
-    <joint name="arm_one_link_1_joint" type="revolute">
+    <joint name="arm_one_link_1_joint" type="fixed">
         <origin xyz="-0.012653 -0.012654 0.196317" rpy="0 0 0"/>
         <parent link="arm_one_base"/>
@@ -61,5 +61,5 @@
     </gazebo>
     <!--Arm One Link-2-->
-    <joint name="arm_one_link_2_joint" type="continuous">
+    <joint name="arm_one_link_2_joint" type="fixed">
         <origin xyz="0.0 0.0 0.173683" rpy="0 0 0"/>
         <parent link="arm_one_link_1"/>
@@ -90,5 +90,5 @@
     </gazebo>
     <!--Arm One Link-3-->
-    <joint name="arm_one_link_3_joint" type="revolute">
+    <joint name="arm_one_link_3_joint" type="fixed">
         <origin xyz="0.0 0.0 0.173684" rpy="0 0 0"/>
         <parent link="arm_one_link_2"/>
@@ -120,5 +120,5 @@
     </gazebo>
     <!--Arm One Link-4-->
-    <joint name="arm_one_link_4_joint" type="continuous">
+    <joint name="arm_one_link_4_joint" type="fixed">
         <origin xyz="-0.086842 0.086842 0.122812" rpy="0 0 0"/>
         <parent link="arm_one_link_3"/>
@@ -149,5 +149,5 @@
     </gazebo>
     <!--Arm One Link-5-->
-    <joint name="arm_one_link_5_joint" type="revolute">
+    <joint name="arm_one_link_5_joint" type="fixed">
         <origin xyz="-0.086842 0.086842 0.122813" rpy="0 0 0"/>
         <parent link="arm_one_link_4"/>
@@ -179,5 +179,5 @@
     </gazebo>
     <!--Arm One Gripper Hand-->
-    <joint name="arm_one_gripper_joint" type="continuous">
+    <joint name="arm_one_gripper_joint" type="fixed">
         <origin xyz="-0.122813 0.122812 0.0" rpy="0 0 0"/>
         <parent link="arm_one_link_5"/>
@@ -208,5 +208,5 @@
     </gazebo>
     <!--Arm One Gripper Finger-1-->
-    <joint name="arm_one_finger_1_joint" type="revolute">
+    <joint name="arm_one_finger_1_joint" type="fixed">
         <origin xyz="-0.042426 0.06364 0.0" rpy="0 0 0"/>
         <parent link="arm_one_gripper_hand"/>
@@ -238,5 +238,5 @@
     </gazebo>
     <!--Arm One Gripper Finger-2-->
-    <joint name="arm_one_finger_2_joint" type="revolute">
+    <joint name="arm_one_finger_2_joint" type="fixed">
         <origin xyz="-0.063639 0.042427 0.0" rpy="0 0 0"/>
         <parent link="arm_one_gripper_hand"/>
@@ -268,5 +268,5 @@
     </gazebo>
     <!--Arm Base Two-->
-    <joint name="arm_two_base_joint" type="continuous">
+    <joint name="arm_two_base_joint" type="fixed">
         <origin xyz="-0.275 0.675 0.07" rpy="0 0 0"/>
         <parent link="basket_link"/>
@@ -297,5 +297,5 @@
     </gazebo>
     <!--Arm Two Link-1-->
-    <joint name="arm_two_link_1_joint" type="revolute">
+    <joint name="arm_two_link_1_joint" type="fixed">
         <origin xyz="0.012653 0.012653 0.196317" rpy="0 0 0"/>
         <parent link="arm_two_base"/>
@@ -327,5 +327,5 @@
     </gazebo>
     <!--Arm Two Link-2-->
-    <joint name="arm_two_link_2_joint" type="continuous">
+    <joint name="arm_two_link_2_joint" type="fixed">
         <origin xyz="0.0 0.0 0.173683" rpy="0 0 0"/>
         <parent link="arm_two_link_1"/>
@@ -356,5 +356,5 @@
     </gazebo>
     <!--Arm Two Link-3-->
-    <joint name="arm_two_link_3_joint" type="revolute">
+    <joint name="arm_two_link_3_joint" type="fixed">
         <origin xyz="0.0 0.0 0.173684" rpy="0 0 0"/>
         <parent link="arm_two_link_2"/>
@@ -386,5 +386,5 @@
     </gazebo>
     <!--Arm Two Link-4-->
-    <joint name="arm_two_link_4_joint" type="continuous">
+    <joint name="arm_two_link_4_joint" type="fixed">
         <origin xyz="0.086842 -0.086842 0.122812" rpy="0 0 0"/>
         <parent link="arm_two_link_3"/>
@@ -415,5 +415,5 @@
     </gazebo>
     <!--Arm Two Link-5-->
-    <joint name="arm_two_link_5_joint" type="revolute">
+    <joint name="arm_two_link_5_joint" type="fixed">
         <origin xyz="0.086842 -0.086842 0.122813" rpy="0 0 0"/>
         <parent link="arm_two_link_4"/>
@@ -445,5 +445,5 @@
     </gazebo>
     <!--Arm Two Gripper Hand-->
-    <joint name="arm_two_gripper_joint" type="continuous">
+    <joint name="arm_two_gripper_joint" type="fixed">
         <origin xyz="0.122813 -0.122812 0.0" rpy="0 0 0"/>
         <parent link="arm_two_link_5"/>
@@ -474,5 +474,5 @@
     </gazebo>
     <!--Arm Two Gripper Finger-1-->
-    <joint name="arm_two_finger_1_joint" type="revolute">
+    <joint name="arm_two_finger_1_joint" type="fixed">
         <origin xyz="0.063639 -0.042427 -0.0075" rpy="0 0 0"/>
         <parent link="arm_two_gripper_hand"/>
@@ -504,5 +504,5 @@
     </gazebo>
     <!--Arm Two Gripper Finger-2-->
-    <joint name="arm_two_finger_2_joint" type="revolute">
+    <joint name="arm_two_finger_2_joint" type="fixed">
         <origin xyz="0.042426 -0.06364 -0.0075" rpy="0 0 0"/>
         <parent link="arm_two_gripper_hand"/>
