Commit message: added front and right cameras

File: mobile_manipulator/description/sensors/cameras.xacro (robot description, xacro)
@@ -1,3 +1,87 @@
 <?xml version="1.0"?>
 <robot xmlns:xacro="http://www.ros.org/wiki/xacro" name="robot">
+    <!--Front Camera-->
+    <joint name="front_camera_joint" type="fixed">
+        <origin xyz="0 0.71 0.1" rpy="0 0 0"/>
+        <parent link="basket_link"/>
+        <child link="front_camera_link"/>
+    </joint>
+    <link name="front_camera_link">
+        <visual>
+            <geometry>
+                <box size="0.06 0.01 0.03"/>
+            </geometry>
+        </visual>
+    </link>
+    <joint name="front_camera_optical_joint" type="fixed">
+        <origin xyz="0 0 0" rpy="${-pi/2} 0 0"/> <!--${-pi/2} 0 ${-pi/2}"-->
+        <parent link="front_camera_link"/>
+        <child link="front_camera_link_optical"/>
+    </joint>
+    <link name="front_camera_link_optical"> </link>
+    <gazebo reference="front_camera_link">
+        <material>Gazebo/Black</material>
+        <sensor type="depth" name="front_camera">
+            <visualize>true</visualize>
+            <update_rate>10</update_rate>
+            <camera>
+                <pose>0 0 0 0 0 1.57</pose>
+                <horizontal_fov>1.089</horizontal_fov>
+                <image>
+                    <width>640</width>
+                    <height>480</height>
+                    <format>B8G8R8</format>
+                </image>
+                <clip>
+                    <near>0.05</near>
+                    <far>8.0</far>
+                </clip>
+            </camera>
+            <plugin name="front_camera_controller" filename="libgazebo_ros_camera.so">
+                <frame_name>front_camera_link_optical</frame_name>
+            </plugin>
+        </sensor>
+    </gazebo>
+    <!--Right Camera-->
+    <joint name="right_camera_joint" type="fixed">
+        <origin xyz="0.31 0 0.1" rpy="0 0 0"/>
+        <parent link="basket_link"/>
+        <child link="right_camera_link"/>
+    </joint>
+    <link name="right_camera_link">
+        <visual>
+            <geometry>
+                <box size="0.01 0.06 0.03"/>
+            </geometry>
+        </visual>
+    </link>
+    <joint name="right_camera_optical_joint" type="fixed">
+        <origin xyz="0 0 0" rpy="${-pi/2} 0 ${-pi/2}"/> <!--${-pi/2} 0 ${-pi/2}"-->
+        <parent link="right_camera_link"/>
+        <child link="right_camera_link_optical"/>
+    </joint>
+    <link name="right_camera_link_optical"> </link>
+    <gazebo reference="right_camera_link">
+        <material>Gazebo/Black</material>
+        <sensor type="depth" name="right_camera">
+            <visualize>true</visualize>
+            <update_rate>10</update_rate>
+            <camera>
+                <pose>0 0 0 0 0 0</pose>
+                <horizontal_fov>1.089</horizontal_fov>
+                <image>
+                    <width>640</width>
+                    <height>480</height>
+                    <format>B8G8R8</format>
+                </image>
+                <clip>
+                    <near>0.05</near>
+                    <far>8.0</far>
+                </clip>
+            </camera>
+            <plugin name="right_camera_controller" filename="libgazebo_ros_camera.so">
+                <frame_name>right_camera_link_optical</frame_name>
+            </plugin>
+        </sensor>
+    </gazebo>
 </robot>

Commit message: completed adding 3 cameras to the cart

File: mobile_manipulator/description/sensors/cameras.xacro (robot description, xacro)
@@ -27,7 +27,7 @@
             <camera>
                 <pose>0 0 0 0 0 1.57</pose>
-                <horizontal_fov>1.089</horizontal_fov>
+                <horizontal_fov>1.8</horizontal_fov>
                 <image>
-                    <width>640</width>
+                    <width>800</width>
                     <height>480</height>
                     <format>B8G8R8</format>
@@ -69,7 +69,7 @@
             <camera>
                 <pose>0 0 0 0 0 0</pose>
-                <horizontal_fov>1.089</horizontal_fov>
+                <horizontal_fov>1.8</horizontal_fov>
                 <image>
-                    <width>640</width>
+                    <width>800</width>
                     <height>480</height>
                     <format>B8G8R8</format>
@@ -85,3 +85,45 @@
         </sensor>
     </gazebo>
+    <!--Left Camera-->
+    <joint name="left_camera_joint" type="fixed">
+        <origin xyz="-0.31 0 0.1" rpy="0 0 0"/>
+        <parent link="basket_link"/>
+        <child link="left_camera_link"/>
+    </joint>
+    <link name="left_camera_link">
+        <visual>
+            <geometry>
+                <box size="0.01 0.06 0.03"/>
+            </geometry>
+        </visual>
+    </link>
+    <joint name="left_camera_optical_joint" type="fixed">
+        <origin xyz="0 0 0" rpy="${-pi/2} 0 ${pi/2}"/> <!--${-pi/2} 0 ${-pi/2}"-->
+        <parent link="left_camera_link"/>
+        <child link="left_camera_link_optical"/>
+    </joint>
+    <link name="left_camera_link_optical"> </link>
+    <gazebo reference="left_camera_link">
+        <material>Gazebo/Black</material>
+        <sensor type="depth" name="left_camera">
+            <visualize>true</visualize>
+            <update_rate>10</update_rate>
+            <camera>
+                <pose>0 0 0 0 0 3.14</pose>
+                <horizontal_fov>1.8</horizontal_fov>
+                <image>
+                    <width>800</width>
+                    <height>480</height>
+                    <format>B8G8R8</format>
+                </image>
+                <clip>
+                    <near>0.05</near>
+                    <far>8.0</far>
+                </clip>
+            </camera>
+            <plugin name="left_camera_controller" filename="libgazebo_ros_camera.so">
+                <frame_name>left_camera_link_optical</frame_name>
+            </plugin>
+        </sensor>
+    </gazebo>
 </robot>
